File: Circuit/Circuit.kicad_sch (KiCad schematic)
At the start: 16 parts, among them J1 Conn_01x20, J2 Conn_01x20, U1 TL072, U2 AMS1117-3.3, Y1 Crystal

Commit message: final PCB design done
Parts:
- removed BoostConverter1: Conn_01x02, Connector_JST:JST_EH_B2B-EH-A_1x02_P2.50mm_Vertical, symbol Connector_Generic:Conn_01x02
- added C3: 10nF, Capacitor_THT:C_Disc_D5.0mm_W2.5mm_P5.00mm, symbol Device:C
- added MuscleSensor_PowerInput2: Conn_01x03, Connector_JST:JST_EH_S3B-EH_1x03_P2.50mm_Horizontal, symbol Connector_Generic:Conn_01x03
- C2: footprint (none) -> Capacitor_THT:CP_Radial_D8.0mm_P3.80mm
Connections:
- net +12V: now also C2.1
- net +24V: now also MuscleSensor_PowerInput2.3 (Pin_3); no longer C2.1
- net +3.3V: now also J2.5 (Pin_5), C3.1; no longer J2.16 (Pin_16)
- net GND: now also C2.2, J2.3 (Pin_3), C3.2; no longer J2.18 (Pin_18)
- net GNDA: now also MuscleSensor_PowerInput2.1 (Pin_1); no longer C2.2
- net Servo1: now also J2.15 (Pin_15); no longer J2.6 (Pin_6)
- net Servo2: now also J2.16 (Pin_16); no longer J2.5 (Pin_5)
- net Servo3: now also J2.18 (Pin_18); no longer J2.3 (Pin_3)
- net Servo4: now also J2.19 (Pin_19); no longer J2.2 (Pin_2)
- net Servo5: now also J2.20 (Pin_20); no longer J2.1 (Pin_1)
- net at MuscleSensor_PowerInput1.2 (Pin_2), R1.2, R2.1: now also MuscleSensor_PowerInput2.2 (Pin_2)
Other:
- moved on the sheet: C2, J2, MuscleSensor_PowerInput1, R1, R2, U1C

Commit message: BOM done and minor changes
Parts:
- removed C1: C, symbol Device:C
Changed lines of the file:
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@@
   (junction (at 177.8 60.96) (diameter 0) (color 0 0 0 0)
   )
-  (junction (at 100.33 88.9) (diameter 0) (color 0 0 0 0)
-  )
   (junction (at 57.15 81.28) (diameter 0) (color 0 0 0 0)
   )
@@
   (junction (at 215.9 118.11) (diameter 0) (color 0 0 0 0)
   )
-  (junction (at 109.22 81.28) (diameter 0) (color 0 0 0 0)
-  )
   (junction (at 215.9 100.33) (diameter 0) (color 0 0 0 0)
   )
@@
   )
   (wire (pts (xy 177.8 76.2) (xy 168.91 76.2))
-    (stroke (width 0) (type default))
-  )
-  (wire (pts (xy 100.33 88.9) (xy 109.22 88.9))
     (stroke (width 0) (type default))
   )
@@
         )
       )
-    )
-  )
-  (symbol (lib_id "Device:C") (at 109.22 85.09 180) (unit 1)
-    (in_bom yes) (on_board yes) (dnp no)
-    (property "Reference" "C1" (at 111.76 83.82 0)
-      (effects (font (size 1.27 1.27)) (justify right))
-    )
-    (property "Value" "C" (at 111.76 86.36 0)
-      (effects (font (size 1.27 1.27)) (justify right))
-    )
-    (property "Footprint" "" (at 108.2548 81.28 0)
-      (effects (font (size 1.27 1.27)) hide)
-    )
-    (property "Datasheet" "~" (at 109.22 85.09 0)
-      (effects (font (size 1.27 1.27)) hide)
-    )
-    (pin "2")
-    (pin "1")
-    (instances
-      (project "Circuit"
-        (path "/8d3eb525-272e-499d-b633-4178066a4d6b"
-          (reference "C1") (unit 1)
-        )
-      )
